File: bkm-68x-simple.kicad_sch (KiCad schematic)
At the start: 2 parts

Commit message: Initial BKM-68Xtreme fork
Parts:
- H1, H2: value (none) -> Keystone 7794; footprint (none) -> keystone-7794:7794-X
