File: bkm-68x-video.kicad_sch (KiCad schematic)
At the start: 86 parts

Commit message: Initial BKM-68Xtreme fork
Parts:
- removed D7, D8: (no value), symbol bkm-68x-simple-rescue:D_Small_ALT
- removed J13, J14, J15, J16, J17, J22, J4: (no value), symbol bkm-68x-simple-rescue:Conn_Coaxial
- removed R4: (no value), symbol bkm-68x-simple-rescue:R
- removed SW3, SW4, SW5, SW6, SW7: (no value), symbol Switch:SW_DPDT_x2
- added C901, C902, C903, C904, C905, C911, C912, C913, C914, C915, C961, C962, C963, C964: 0.1uF, Capacitor_SMD:C_0805_2012Metric_Pad1.18x1.45mm_HandSolder, symbol bkm-68x-simple-rescue:C_Small
- added J901: SCART-F, ninigi-scart-ra:NINIGI-SCART-RA, symbol Connector:SCART-F
- added J902: AUDIO_L_OUT, rcj-41x:RCJ-04X, symbol bkm-68x-simple-rescue:Conn_Coaxial
- added J903: AUDIO_R_OUT, rcj-41x:RCJ-04X, symbol bkm-68x-simple-rescue:Conn_Coaxial
- added J911: DB15_Female_HighDensity_MountingHoles, hd15-vga:HD15-VGA, symbol Connector:DB15_Female_HighDensity_MountingHoles
- added R901, R902, R903, R904, R911, R912, R913, R914: 75R, Resistor_SMD:R_0805_2012Metric_Pad1.20x1.40mm_HandSolder, symbol bkm-68x-simple-rescue:R
- added U901, U911: THS7374, Package_SO:TSSOP-14_4.4x5mm_P0.65mm, symbol ths7374:THS7374
- added U961, U962, U963, U964: TS5A3359DCU, Package_SO:VSSOP-8_2.4x2.1mm_P0.5mm, symbol ts5a3359:TS5A3359DCU
- C1, C10, C13, C2, C27, C3, C4, C5, C6, C62, C63, C64, C7, C9: value (none) -> 0.1uF; footprint (none) -> Capacitor_SMD:C_0805_2012Metric_Pad1.18x1.45mm_HandSolder
- C11: value (none) -> 56nF; footprint (none) -> Capacitor_SMD:C_0805_2012Metric_Pad1.18x1.45mm_HandSolder
- C30, C31, C32, C69: value (none) -> NM; footprint (none) -> Capacitor_SMD:C_0805_2012Metric_Pad1.18x1.45mm_HandSolder
- C33: value (none) -> 22pF; footprint (none) -> Capacitor_SMD:C_0805_2012Metric_Pad1.18x1.45mm_HandSolder
- C54: value (none) -> 100pF; footprint (none) -> Capacitor_SMD:C_0805_2012Metric_Pad1.18x1.45mm_HandSolder
- C55: value (none) -> 470pF; footprint (none) -> Capacitor_SMD:C_0805_2012Metric_Pad1.18x1.45mm_HandSolder
- C65: value (none) -> 220pF; footprint (none) -> Capacitor_SMD:C_0805_2012Metric_Pad1.18x1.45mm_HandSolder
- D1, D10, D2, D3, D4, D5, D6, D9: value (none) -> NM; footprint (none) -> Diode_SMD:D_SOD-123
- J1: value (none) -> PR_R; footprint (none) -> rcj-41x:RCJ-04X
- J10: value (none) -> TP_VIDEO_OE; footprint (none) -> TestPoint:TestPoint_Pad_D2.0mm
- J11: value (none) -> TP_VSYNC; footprint (none) -> TestPoint:TestPoint_Pad_D2.0mm
- J2: value (none) -> Y_G; footprint (none) -> rcj-41x:RCJ-04X
- J3: value (none) -> PB_B; footprint (none) -> rcj-41x:RCJ-04X
- J5: value (none) -> TP_Y_G; footprint (none) -> TestPoint:TestPoint_Pad_D2.0mm
- J6: value (none) -> TP_PB_B; footprint (none) -> TestPoint:TestPoint_Pad_D2.0mm
- J7: value (none) -> TP_PR_R; footprint (none) -> TestPoint:TestPoint_Pad_D2.0mm
- J8: value (none) -> TP_HSYNC; footprint (none) -> TestPoint:TestPoint_Pad_D2.0mm
- J9: value (none) -> TP_INT_EXT_SYNC; footprint (none) -> TestPoint:TestPoint_Pad_D2.0mm
- Q1, Q2: value (none) -> MMBT3904; footprint (none) -> Package_TO_SOT_SMD:SOT-23_Handsoldering
- R1, R10, R12, R14, R2, R3, R6: value (none) -> 75R; footprint (none) -> Resistor_SMD:R_0805_2012Metric_Pad1.20x1.40mm_HandSolder
- R11, R13, R9: value (none) -> 150R; footprint (none) -> Resistor_SMD:R_0805_2012Metric_Pad1.20x1.40mm_HandSolder
- R44, R7: value (none) -> 1K; footprint (none) -> Resistor_SMD:R_0805_2012Metric_Pad1.20x1.40mm_HandSolder
- R71, R72: value (none) -> 47R; footprint (none) -> Resistor_SMD:R_0805_2012Metric_Pad1.20x1.40mm_HandSolder
- R8, R81, R84: value (none) -> 10K; footprint (none) -> Resistor_SMD:R_0805_2012Metric_Pad1.20x1.40mm_HandSolder
- R80: value (none) -> 100R; footprint (none) -> Resistor_SMD:R_0805_2012Metric_Pad1.20x1.40mm_HandSolder
- R89: value (none) -> NM; footprint (none) -> Resistor_SMD:R_0805_2012Metric_Pad1.20x1.40mm_HandSolder
- R90: value (none) -> 0R; footprint (none) -> Resistor_SMD:R_0805_2012Metric_Pad1.20x1.40mm_HandSolder
- U1: value (none) -> ADG1611BCPZ; footprint (none) -> Package_CSP:LFCSP-16-1EP_4x4mm_P0.65mm_EP2.4x2.4mm
- U16: value (none) -> SN74LVC1G14DBV; footprint (none) -> Package_TO_SOT_SMD:SOT-23-5
- U17: value (none) -> ISL4089; footprint (none) -> Package_SO:SOIC-8_3.9x4.9mm_P1.27mm; JLC (none) -> SOIC-8; LCSC (none) -> C2649399
- U2: value (none) -> THS7374; footprint (none) -> Package_SO:TSSOP-14_4.4x5mm_P0.65mm
- U3: value (none) -> ISL59885; footprint (none) -> Package_SO:SOIC-8_3.9x4.9mm_P1.27mm
- U301: value (none) -> FSA2257MUX; footprint (none) -> Package_SO:MSOP-10_3x3mm_P0.5mm; JLC (none) -> MSOP-10; LCSC (none) -> C894842
- U501: value (none) -> ADG1611; footprint (none) -> Package_SO:TSSOP-16_4.4x5mm_P0.65mm
- U8: value (none) -> TC7WH125; footprint (none) -> Package_SO:SSOP-8_2.95x2.8mm_P0.65mm
Connections:
- net EXT_SYNC_IN is gone; now on net GND: C6.2
- net PB_B_IN is gone; now on net PB_IN: C5.2, D3.2 (A), D4.1 (K), J3.1 (In)
- net PR_R_IN is gone; now on net PR_IN: C3.2, D5.2 (A), D6.1 (K), J1.1 (In)
- net Y_G_IN is gone; now on net Y_IN: C4.2, D1.2 (A), D2.1 (K), J2.1 (In)
- net +5VA: now also C905.2, C915.2, C961.2, C962.2, C963.2, C964.2, U901.10 (VCC), U901.9 (BYPASS), U911.10 (VCC), U911.9 (BYPASS), U961.8 (VCC), U962.8 (VCC), U963.8 (VCC), U964.8 (VCC)
- net EXT_SYNC_AMP: now also U964.7 (COM); no longer U2.11 (CH4_OUT)
- net GND: now also C905.1, C915.1, C961.1, C962.1, C963.1, C964.1, J901.13 (P13), J901.14 (P14), J901.17 (P17), J901.18 (P18), J901.21 (P21), J901.4 (P4), J901.5 (P5), J901.9 (P9), J902.2 (Ext), J903.2 (Ext), J911.0, J911.10, J911.5, J911.6, J911.7, J911.8, R901.1, R902.1, R903.1, R904.1, R911.1, R912.1, R913.1, R914.1, U901.5 (GND), U901.6 (DISABLE), U911.5 (GND), U911.6 (DISABLE), U961.4 (GND), U962.4 (GND), U963.4 (GND), U964.1 (NO0), U964.4 (GND)
- net PB_B_AMP: now also U963.7 (COM); no longer U2.12 (CH3_OUT)
- net PR_R_AMP: now also U961.7 (COM); no longer U2.14 (CH1_OUT)
- net Y_G_AMP: now also U962.7 (COM); no longer U2.13 (CH2_OUT)
- net Y_IN: now reaches R1.1
- net PR_IN: now reaches R3.1
- net PB_IN: now reaches R2.1
- net VSYNC_VGA_IN: now reaches D10.1 (K), D9.2 (A), R8.1
- net VSYNC_VGA_IN: now also R6.1, J911.14
- new net: C903.1, U901.3 (CH3_IN)
- new net: C901.1, U901.1 (CH1_IN)
- new net: C902.1, U901.2 (CH2_IN)
- new net: C904.1, U901.4 (CH4_IN)
- new net: C913.1, U911.3 (CH3_IN)
- new net: C912.1, U911.2 (CH2_IN)
- new net: C911.1, U911.1 (CH1_IN)
- new net: C914.1, U911.4 (CH4_IN)
- new net B_SCART_AMP: U901.12 (CH3_OUT), U963.2 (NO1)
- new net B_SCART_IN: C903.2, J901.7 (P7), R903.2
- new net B_VGA_AMP: U911.14 (CH1_OUT), U963.3 (NO2)
- new net B_VGA_IN: C911.2, J911.3, R913.2
- new net CSYNC_SCART_IN: C904.2, J901.20 (P20), R904.2
- new net G_SCART_AMP: U901.13 (CH2_OUT), U962.2 (NO1)
- new net G_SCART_IN: C902.2, J901.11 (P11), R902.2
- new net G_VGA_AMP: U911.13 (CH2_OUT), U962.3 (NO2)
- new net G_VGA_IN: C912.2, J911.2, R912.2
- new net HCSYNC_VGA_AMP: U911.11 (CH4_OUT), U964.3 (NO2)
- new net HCSYNC_VGA_IN: C914.2, J911.13, R914.2
- new net PB_AMP: U2.12 (CH3_OUT), U963.1 (NO0)
- new net PR_AMP: U2.14 (CH1_OUT), U961.1 (NO0)
- new net R_SCART_AMP: U901.14 (CH1_OUT), U961.2 (NO1)
- new net R_SCART_IN: C901.2, J901.15 (P15), R901.2
- new net R_VGA_AMP: U911.12 (CH3_OUT), U961.3 (NO2)
- new net R_VGA_IN: C913.2, J911.1, R911.2
- new net SCART_AUDIO_L: J901.6 (P6), J902.1 (In)
- new net SCART_AUDIO_R: J901.2 (P2), J903.1 (In)
- new net SCART_BLANK_IN: J901.16 (P16)
- new net SRC_SEL1: U961.6 (IN1), U962.6 (IN1), U963.6 (IN1), U964.6 (IN1)
- new net SRC_SEL2: U961.5 (IN2), U962.5 (IN2), U963.5 (IN2), U964.5 (IN2)
- new net SYNC_SCART_AMP: U901.11 (CH4_OUT), U964.2 (NO1)
- new net VGA_5V_IN: J911.9
- new net Y_AMP: U2.13 (CH2_OUT), U962.1 (NO0)
- no-connect marks 2 -> 13
Other:
- moved on the sheet: C10, C11, C13, C27, C3, C33, C4, C5, C54, C55, C6, C62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
