File: connectors.kicad_sch (KiCad schematic)
At the start: 3 parts

Commit message: Initial BKM-68Xtreme fork
Parts:
- CN985, CN986: value (none) -> mezz-conn-02x50; footprint (none) -> TX24-100R-LT-H1E:TX24-100R-LT-H1E
- J12: value (none) -> JTAG; footprint (none) -> Connector_PinHeader_2.54mm:PinHeader_1x05_P2.54mm_Vertical
