File: fpga.kicad_sch (KiCad schematic)
At the start: 126 parts

Commit message: Initial BKM-68Xtreme fork
Parts:
- added R4, R45: 22R, Resistor_SMD:R_0805_2012Metric_Pad1.20x1.40mm_HandSolder, symbol bkm-68x-simple-rescue:R
- added unit 6 of U7
- C12, C20, C21, C22, C71, C8: value (none) -> 0.1uF; footprint (none) -> Capacitor_SMD:C_0805_2012Metric_Pad1.18x1.45mm_HandSolder
- C401, C402, C403, C404: value (none) -> 10pF; footprint (none) -> Capacitor_SMD:C_0603_1608Metric_Pad1.08x0.95mm_HandSolder
- C601, C602, C851, C852, C853, C854, C855, C856, C857, C858, C859, C860, C861, C862: value (none) -> 0.1uF; footprint (none) -> Capacitor_SMD:C_0603_1608Metric_Pad1.08x0.95mm_HandSolder
- C831: value (none) -> 10uF; footprint (none) -> Capacitor_SMD:C_0805_2012Metric_Pad1.18x1.45mm_HandSolder
- D13: value (none) -> DEBUG1; footprint (none) -> LED_SMD:LED_0805_2012Metric_Pad1.15x1.40mm_HandSolder
- D14: value (none) -> DEBUG2; footprint (none) -> LED_SMD:LED_0805_2012Metric_Pad1.15x1.40mm_HandSolder
- D401, D402, D403, D404: value (none) -> NM; footprint (none) -> Diode_SMD:D_SOD-123
- J19: renamed from J?; value (none) -> TP_NORM_Y_G; footprint (none) -> TestPoint:TestPoint_Pad_D2.0mm
- J20: renamed from J?; value (none) -> TP_RGB_COMP_X; footprint (none) -> TestPoint:TestPoint_Pad_D2.0mm
- J21: renamed from J?; value (none) -> TP_HD_SD_X; footprint (none) -> TestPoint:TestPoint_Pad_D2.0mm
- J401: value (none) -> JTAG; footprint (none) -> Connector_PinHeader_2.54mm:PinHeader_2x05_P2.54mm_Vertical
- J601: value (none) -> SPI_PROG; footprint (none) -> Connector_PinHeader_2.54mm:PinHeader_1x07_P2.54mm_Vertical
- R15, R16, R17, R18, R19, R20, R21, R22, R23, R25, R36, R38, R42, R43, R5: value (none) -> 68R; footprint (none) -> Resistor_SMD:R_0805_2012Metric_Pad1.20x1.40mm_HandSolder
- R24, R26, R27, R28, R29, R30, R31, R32: value (none) -> 47R; footprint (none) -> Resistor_SMD:R_0805_2012Metric_Pad1.20x1.40mm_HandSolder
- R33, R34, R35, R39: value (none) -> 47K; footprint (none) -> Resistor_SMD:R_0805_2012Metric_Pad1.20x1.40mm_HandSolder
- R37: value (none) -> 22K; footprint (none) -> Resistor_SMD:R_0805_2012Metric_Pad1.20x1.40mm_HandSolder
- R40, R41, R78, R79, R87, R88: value (none) -> 22R; footprint (none) -> Resistor_SMD:R_0805_2012Metric_Pad1.20x1.40mm_HandSolder
- R401, R402, R403, R404, R801, R802, R803, R804, R805, R806, R807, R831: value (none) -> 10K; footprint (none) -> Resistor_SMD:R_0603_1608Metric_Pad0.98x0.95mm_HandSolder
- R405: value (none) -> 1K; footprint (none) -> Resistor_SMD:R_0603_1608Metric_Pad0.98x0.95mm_HandSolder
- R46, R601, R602, R77: value (none) -> 10K; footprint (none) -> Resistor_SMD:R_0805_2012Metric_Pad1.20x1.40mm_HandSolder
- R47, R48, R49, R50, R51, R52, R53, R62, R63, R64, R65, R66, R67: renamed from R?; value (none) -> 68R; footprint (none) -> Resistor_SMD:R_0805_2012Metric_Pad1.20x1.40mm_HandSolder
- R54, R55, R56, R57, R58, R59, R60, R61, R68, R69, R70: renamed from R?; value (none) -> 22R; footprint (none) -> Resistor_SMD:R_0805_2012Metric_Pad1.20x1.40mm_HandSolder
- R82: renamed from R?; value (none) -> 470R; footprint (none) -> Resistor_SMD:R_0805_2012Metric_Pad1.20x1.40mm_HandSolder
- R820: value (none) -> 22R; footprint (none) -> Resistor_SMD:R_0603_1608Metric_Pad0.98x0.95mm_HandSolder
- R83: renamed from R?; value (none) -> 390R; footprint (none) -> Resistor_SMD:R_0805_2012Metric_Pad1.20x1.40mm_HandSolder
- SW1, SW2: value (none) -> FORCE_VIDEO; footprint (none) -> Button_Switch_SMD:SW_SPST_EVQP7C
- U10: value (none) -> 74LVC541A; footprint (none) -> Package_SO:TSSOP-20_4.4x6.5mm_P0.65mm
- U11, U19: value (none) -> 74LVC2G34; footprint (none) -> Package_TO_SOT_SMD:SOT-23-6_Handsoldering
- U12: value (none) -> TC7SZ125FU; footprint (none) -> Package_TO_SOT_SMD:SOT-353_SC-70-5_Handsoldering
- U5, U6, U7: value (none) -> 74LVC14A; footprint (none) -> Package_SO:TSSOP-14_4.4x5mm_P0.65mm
- U601: value (none) -> W25Q128JVS; footprint (none) -> Package_SO:SOIC-8_5.23x5.23mm_P1.27mm
- U801: value (none) -> T8Q144; footprint (none) -> Package_QFP:TQFP-144_20x20mm_P0.5mm
- U9: value (none) -> KC2520Z50; footprint (none) -> Oscillator:Oscillator_SMD_Kyocera_KC2520Z-4Pin_2.5x2.0mm
Connections:
- net +3.3V: now also U7.14 (VCC)
- net GND: now also U801.46 (GPIOB_TXN06), U7.13, U7.7 (GND)
- net at U801.55 (GPIOB_RXP00): now also R45.1
- net at U801.65 (GPIOB_RXN07): now also R4.1
- net HWID1: now reaches U801.47 (GPIOB_TXP08)
- new net SRC_SEL1: R4.2
- new net SRC_SEL2: R45.2
- no-connect marks 59 -> 57
