File: power-supply.kicad_sch (KiCad schematic)
At the start: 48 parts

Commit message: Initial BKM-68Xtreme fork
Parts:
- C111, C112, C113, C114, C23: value (none) -> 1uF; footprint (none) -> Capacitor_SMD:C_0805_2012Metric_Pad1.18x1.45mm_HandSolder
- C14, C16, C18, C61: value (none) -> 100uF; footprint (none) -> Capacitor_SMD:CP_Elec_6.3x5.3
- C15, C17, C19, C56, C57, C59: value (none) -> 0.1uF; footprint (none) -> Capacitor_SMD:C_0805_2012Metric_Pad1.18x1.45mm_HandSolder
- C24, C58: value (none) -> 100uF; footprint (none) -> Capacitor_SMD:CP_Elec_6.3x5.4
- C25, C28, C68, C70: value (none) -> 10uF; footprint (none) -> Capacitor_SMD:C_0805_2012Metric_Pad1.18x1.45mm_HandSolder
- C26: value (none) -> 330uF/LOW_ESR; footprint (none) -> Capacitor_SMD:CP_Elec_6.3x7.7
- C801, C802, C803, C804, C805, C806, C807, C808, C809, C810, C811, C812: value (none) -> 0.1uF; footprint (none) -> Capacitor_SMD:C_0603_1608Metric_Pad1.08x0.95mm_HandSolder
- J101: value (none) -> TP_1V2; footprint (none) -> TestPoint:TestPoint_Pad_D2.0mm
- J102: value (none) -> TP_3V3; footprint (none) -> TestPoint:TestPoint_Pad_D2.0mm
- J103: value (none) -> TP_GNDD1; footprint (none) -> TestPoint:TestPoint_Pad_D2.0mm
- J18: value (none) -> Conn_01x02_Male; footprint (none) -> Connector_PinHeader_2.54mm:PinHeader_1x02_P2.54mm_Vertical
- J201: value (none) -> TP_NEG5V; footprint (none) -> TestPoint:TestPoint_Pad_D2.0mm
- J202: value (none) -> TP_5V; footprint (none) -> TestPoint:TestPoint_Pad_D2.0mm
- J203: value (none) -> TP_GNDA1; footprint (none) -> TestPoint:TestPoint_Pad_D2.0mm
- R101: value (none) -> 10K; footprint (none) -> Resistor_SMD:R_0805_2012Metric_Pad1.20x1.40mm_HandSolder
- U101: value (none) -> NCV8164ASN120T1G; footprint (none) -> Package_SO:TSOP-5_1.65x3.05mm_P0.95mm
- U102: value (none) -> BD33HC0WEFJ-E2; footprint (none) -> Package_SO:HTSOP-8-1EP_3.9x4.9mm_P1.27mm_EP2.4x3.2mm_ThermalVias
- U13: value (none) -> LM2990SX-5.0; footprint (none) -> Package_TO_SOT_SMD:TO-263-3_TabPin2
- U14: value (none) -> BA50BC0FP-E2; footprint (none) -> Package_TO_SOT_SMD:TO-252-3_TabPin2
- U801: value (none) -> T8Q144; footprint (none) -> Package_QFP:TQFP-144_20x20mm_P0.5mm
